File: eagle/low-gain-radio.sch (EAGLE design)
At the start: 127 parts, among them U1 MKW01Z128, U2 SKY65116, U3 W25Q80DV, U4 LP5907MFX-3.3, U6 LP5907MFX-3.3, U7 LD39200, U8 MAAL-010704, Y1 32MHz

Commit message: New OreSat card v0.4 layout, meant for internal backplane positioning. Moved to MMCX conncectors. Routed RF reflectometer lines, moved stuff around to get better access to the RF-RESET, and touched up the new zero ohm resistors in all of the power lines.
Parts:
- added C58: 10nF, rcl_custom:C-EU0603-B-NOSILK
- added CF2: CON-MMCX-F-MOLEX-0734151001, oresat-eagle:CON-MMCX-F-MOLEX-0734151001
- added RF-RESET: TEST-POINT, Tova:TEST-POINT
Connections:
- removed net N$11: R17.1, U6.VOUT
- new net N$12: C39.2, R15.1, R5.2, U4.VIN
- net 3.3V: now also C41.2, C53.1, U4.VOUT; no longer R15.2
- net DC_OUT: now also CF2.CENTER
- net N$6: now also C13.2, R16.1, U7.IN; no longer C41.2, C53.1, R15.1, U4.VOUT
- net N$9: now also C36.2, R17.1, U6.VIN; no longer R16.1, U7.OUT
- net RF_GND: now also C58.1, CF2.SHIELD
- net RF_RESET: now also RF-RESET.1
- net V+: now also R15.2, R16.2, R17.2; no longer C13.2, C36.2, C39.2, R5.2, U$9.VDD, U4.VIN, U6.VIN, U7.IN
- net VBIAS: now also C58.2, U$9.VDD, U6.VOUT; no longer R17.2
- net VPA: now also U7.OUT; no longer R16.2
Other:
- moved on the sheet: C36, C38, C53, R15, R16, R17
